File: Slab.kicad_sch (KiCad schematic)
At the start: 369 parts, among them J1 Conn_01x04, SW1 RotaryEncoder_Switch, U1 Seeeduino Xiao rp2040, U2 PCA9555PW, U3 SN74AHCT125PWR

Commit message: feat: update schematic symbols
Parts:
- LED76, LED77, LED78, LED79, LED80, LED81, LED82, LED83, LED84, LED85, LED86, LED87, LED88, LED89, LED90: footprint PCM_marbastlib-various:LED_6028R -> CustomKeyboardLibrary:LED_6028R_Custom
- U3: footprint CustomKeyboardLibrary:PW14 -> CustomKeyboardLibrary:SN74AHCT125PWR
Changed lines of the file:
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@@
 			)
 		)
-		(property "Footprint" "PCM_marbastlib-various:LED_6028R"
+		(property "Footprint" "CustomKeyboardLibrary:LED_6028R_Custom"
 			(at 153.67 262.89 0)
 			(effects
@@
 			)
 		)
-		(property "Footprint" "PCM_marbastlib-various:LED_6028R"
+		(property "Footprint" "CustomKeyboardLibrary:LED_6028R_Custom"
 			(at 168.91 262.89 0)
 			(effects
@@
 			)
 		)
-		(property "Footprint" "CustomKeyboardLibrary:PW14"
+		(property "Footprint" "CustomKeyboardLibrary:SN74AHCT125PWR"
 			(at 17.78 205.74 0)
 			(effects
@@
 			)
 		)
-		(property "Footprint" "PCM_marbastlib-various:LED_6028R"
+		(property "Footprint" "CustomKeyboardLibrary:LED_6028R_Custom"
 			(at 214.63 262.89 0)
 			(effects
@@
 			)
 		)
-		(property "Footprint" "PCM_marbastlib-various:LED_6028R"
+		(property "Footprint" "CustomKeyboardLibrary:LED_6028R_Custom"
 			(at 62.23 262.89 0)
 			(effects
@@
 			)
 		)
-		(property "Footprint" "PCM_marbastlib-various:LED_6028R"
+		(property "Footprint" "CustomKeyboardLibrary:LED_6028R_Custom"
 			(at 123.19 262.89 0)
 			(effects
@@
 			)
 		)
-		(property "Footprint" "PCM_marbastlib-various:LED_6028R"
+		(property "Footprint" "CustomKeyboardLibrary:LED_6028R_Custom"
 			(at 92.71 262.89 0)
 			(effects
@@
 			)
 		)
-		(property "Footprint" "PCM_marbastlib-various:LED_6028R"
+		(property "Footprint" "CustomKeyboardLibrary:LED_6028R_Custom"
 			(at 77.47 262.89 0)
 			(effects
@@
 			)
 		)
-		(property "Footprint" "PCM_marbastlib-various:LED_6028R"
+		(property "Footprint" "CustomKeyboardLibrary:LED_6028R_Custom"
 			(at 107.95 262.89 0)
 			(effects
@@
 			)
 		)
-		(property "Footprint" "PCM_marbastlib-various:LED_6028R"
+		(property "Footprint" "CustomKeyboardLibrary:LED_6028R_Custom"
 			(at 245.11 262.89 0)
 			(effects
@@
 			)
 		)
-		(property "Footprint" "PCM_marbastlib-various:LED_6028R"
+		(property "Footprint" "CustomKeyboardLibrary:LED_6028R_Custom"
 			(at 138.43 262.89 0)
 			(effects
@@
 			)
 		)
-		(property "Footprint" "PCM_marbastlib-various:LED_6028R"
+		(property "Footprint" "CustomKeyboardLibrary:LED_6028R_Custom"
 			(at 229.87 262.89 0)
 			(effects
@@
 			)
 		)
-		(property "Footprint" "PCM_marbastlib-various:LED_6028R"
+		(property "Footprint" "CustomKeyboardLibrary:LED_6028R_Custom"
 			(at 199.39 262.89 0)
 			(effects
@@
 			)
 		)
-		(property "Footprint" "PCM_marbastlib-various:LED_6028R"
+		(property "Footprint" "CustomKeyboardLibrary:LED_6028R_Custom"
 			(at 184.15 262.89 0)
 			(effects
@@
 			)
 		)
-		(property "Footprint" "PCM_marbastlib-various:LED_6028R"
+		(property "Footprint" "CustomKeyboardLibrary:LED_6028R_Custom"
 			(at 46.99 262.89 0)
 			(effects
@@
 			)
 		)
-		(property "Footprint" "PCM_marbastlib-various:LED_6028R"
+		(property "Footprint" "CustomKeyboardLibrary:LED_6028R_Custom"
 			(at 260.35 262.89 0)
 			(effects

Commit message: feat: init v2 schematic
Parts:
- removed C76, C77, C78, C79, C80, C81, C82, C83, C84, C85, C86, C87, C88, C89, C90: 100nF, Capacitor_SMD:C_1206_3216Metric_Pad1.33x1.80mm_HandSolder, symbol Device:C_Polarized
- removed LED76, LED77, LED78, LED79, LED80, LED81, LED82, LED83, LED84, LED85, LED86, LED87, LED88, LED89, LED90: SK6812MINI-E, CustomKeyboardLibrary:LED_6028R_Custom, symbol PCM_marbastlib-various:SK6812MINI-E
- removed MH1, MH10, MH11, MH12, MH13, MH14, MH15, MH16, MH17, MH18, MH19, MH2, MH20, MH21, MH22, MH23, MH24, MH25, MH26, MH27, MH28, MH29, MH3, MH30, MH4, MH5, MH6, MH7, MH8, MH9: MountingHole_Pad, MountingHole:MountingHole_3.2mm_M3_Pad, symbol Mechanical:MountingHole_Pad
- removed U1: Seeeduino Xiao rp2040, PCM_marbastlib-xp-promicroish:Xiao_rp2040_ACH, symbol PCM_marbastlib-promicroish:Seeeduino_Xiao_rp2040
- added C76, C77, C78, C79, C84: 100nF, symbol Device:C
- added C81, C82: 12pF, symbol Device:C
- added C83, C85: 1uF, symbol Device:C
- added R3, R8: 10k, symbol Device:R
- added R6, R7: 1k, symbol Device:R
- added SW2, SW3: SW_Push, symbol Switch:SW_Push
- added TP1, TP10, TP11, TP12, TP2, TP3, TP4, TP5, TP6, TP7, TP8, TP9: TestPoint, symbol Connector:TestPoint
- added U1: RP2040, Package_DFN_QFN:QFN-56-1EP_7x7mm_P0.4mm_EP3.2x3.2mm, symbol MCU_RaspberryPi:RP2040
- added U4: W25Q128JVS, Package_SO:SOIC-8_5.23x5.23mm_P1.27mm, symbol Memory_Flash:W25Q128JVS
- added U5: AP2112K-3.3, Package_TO_SOT_SMD:SOT-23-5, symbol Regulator_Linear:AP2112K-3.3
- added Y1: 12MHz, symbol Device:Crystal
Connections:
- net +3V3: now also C76.1, C78.1, C79.1, C83.1, R3.1, R8.2, U1.1 (IOVDD), U1.10 (IOVDD), U1.22 (IOVDD), U1.33 (IOVDD), U1.42 (IOVDD), U1.43 (ADC_AVDD), U1.44 (VREG_IN), U1.48 (USB_VDD), U1.49 (IOVDD), U4.8 (VCC), U5.5 (VOUT)
- net +5V: now also C77.1, TP12.1, TP6.1, U5.1 (VIN), U5.3 (EN)
- net GND: now also C76.2, C77.2, C78.2, C79.2, C81.1, C82.1, C83.2, C84.1, C85.1, SW2.2, SW3.2, TP3.1, TP9.1, U1.19 (TESTEN), U1.57 (GND), U4.4 (GND), U5.2 (GND)
- net I2C_1.SCL: no longer R2.2, U2.22 (SCL)
- net I2C_1.SDA: no longer R1.2, U2.23 (SDA)
- net EncoderSwitchOutput renamed EncoderSwitch
- new net: C82.2, U1.20 (XIN), Y1.2
- new net: R7.1, R8.1, U1.56 (QSPI_SS), U4.1 (~{CS})
- new net: TP2.1, U1.25 (SWD)
- new net: C81.2, R6.1, Y1.1
- new net: R6.2, U1.21 (XOUT)
- new net: TP1.1, U1.24 (SWCLK)
- new net: U1.51 (QSPI_SD3), U4.7 (IO3)
- new net: U1.52 (QSPI_SCLK), U4.6 (CLK)
- new net: U1.53 (QSPI_SD0), U4.5 (DI(IO0))
- new net: U1.54 (QSPI_SD2), U4.3 (IO2)
- new net: U1.55 (QSPI_SD1), U4.2 (DO(IO1))
- new net +1V1: C84.2, C85.2, U1.23 (DVDD), U1.45 (VREG_VOUT), U1.50 (DVDD)
- new net BOOT: R7.2, SW2.1
- new net I2C1_SCL: R2.2, TP11.1, U1.5 (GPIO3)
- new net I2C1_SDA: R1.2, TP10.1, U1.4 (GPIO2)
- new net RESET: R3.2, SW3.1, U1.26 (RUN)
- new net UART0_RX: TP5.1, U1.3 (GPIO1)
- new net UART0_TX: TP4.1, U1.2 (GPIO0)
- new net USB_DM: U1.46 (USB_DM)
- new net USB_DP: U1.47 (USB_DP)
Other:
- note added: "128MB QSPI Flash"
- note added: "Boot Switches"
- note added: "Crystal Oscillator"
- note added: "I2C Pullups"
- note added: "Power supply"
- note added: "RP2040"
- note added: "Testpoints 1"
- note added: "Testpoints 2"
- note removed: "Extra LEDs at the top of the keyboard module."
- note removed: "Hot swapable key switches."
- note removed: "I2C Address: 0b0100XXX"
- note removed: "I2C Address: 0b0111100"
- note removed: "I2C IO Expander"
- note removed: "I2C OLED 128x32"
- note removed: "Keys"
- note removed: "LED Bar"
- note removed: "Last 3 digits are decided by A2,A1 and A0. In this case, they are all 0s."
- note removed: "Level shifter from 3.3v to 5v."
- note removed: "Microcontroller"
- note removed: "Mounting holes"
- note removed: "Neopixel RGB LEDs. The last DOUT can be left floating."
- note removed: "OLED display for info and stats. No symbol for it, so generic connector is used instead."
- note removed: "Part: EC11E15244B2"
- note removed: "Pins A0-2 choose the I2C address bits, each can be connected to GND or 3V3."
- note removed: "RGB LEDs"
- note removed: "Rotary Encoder and Switch"
- moved on the sheet: C1, C10, C11, C12, C13, C14, C15, C16, C17, C18, C19, C2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

Commit message: feat: add most parts
Parts:
- removed C1, C10, C11, C12, C13, C14, C15, C16, C17, C18, C19, C2, C20, C21, C22, C23, C24, C25, C26, C27, C28, C29, C3, C30, C31, C32, C33, C34, C35, C36, C37, C38, C39, C4, C40, C41, C42, C43, C44, C45, C46, C47, C48, C49, C5, C50, C51, C52, C53, C54, C55, C56, C57, C58, C59, C6, C60, C61, C62, C63, C64, C65, C66, C67, C68, C69, C7, C70, C71, C72, C73, C74, C75, C8, C9, C91, C96: 100nF, Capacitor_SMD:C_1206_3216Metric_Pad1.33x1.80mm_HandSolder, symbol Device:C_Polarized
- removed D1, D10, D11, D12, D13, D14, D15, D16, D17, D18, D19, D2, D20, D21, D22, D23, D24, D25, D26, D27, D28, D29, D3, D30, D31, D32, D33, D34, D35, D36, D37, D38, D39, D4, D40, D41, D42, D43, D44, D45, D46, D47, D48, D49, D5, D50, D51, D52, D53, D54, D55, D56, D57, D58, D59, D6, D60, D61, D62, D63, D64, D65, D66, D67, D68, D69, D7, D70, D71, D72, D73, D74, D75, D8, D9: 1N4148W, Diode_SMD:D_SOD-123, symbol Diode:1N4148W
- removed MX1: MX_SW_HS, CustomKeyboardLibrary:SW_MX_HS_CPG151101S11_1u_Custom, symbol PCM_marbastlib-mx:MX_SW_HS_CPG151101S11
- removed SW1: RotaryEncoder_Switch, Rotary_Encoder:RotaryEncoder_Alps_EC11E-Switch_Vertical_H20mm, symbol Device:RotaryEncoder_Switch
- added BZ1: Buzzer, symbol Device:Buzzer
- added C1, C10, C11, C12, C13, C14, C15, C16, C17, C18, C19, C2, C20, C21, C22, C23, C24, C25, C26, C27, C28, C29, C3, C30, C31, C32, C33, C34, C35, C36, C37, C38, C39, C4, C40, C41, C42, C43, C44, C45, C46, C47, C48, C49, C5, C50, C51, C52, C53, C54, C55, C56, C57, C58, C59, C6, C60, C61, C62, C63, C64, C65, C66, C67, C68, C69, C7, C70, C71, C72, C73, C74, C75, C8, C80, C86, C87, C88, C89, C9, C90, C91: 100nF, symbol Device:C
- added J2: USB_C_Receptacle_USB2.0_16P, symbol Connector:USB_C_Receptacle_USB2.0_16P
- added LED76: MX_SK6812MINI-E, CustomKeyboardLibrary:LED_MX_6028R-ROT_Custom, symbol PCM_marbastlib-mx:MX_SK6812MINI-E
- added MX15: SW_MX_CHOC, CustomKeyboardLibrary:SW_choc_mx_combined, symbol PCM_marbastlib-mx:MX_SW_HS_CPG151101S11
- added Q1: MMBT3906, Package_TO_SOT_SMD:SOT-23, symbol Transistor_BJT:MMBT3906
- added R10, R11, R4, R5, R9: 10k, symbol Device:R
- added R12, R13: 5.1k, symbol Device:R
- added R14, R15: 27, symbol Device:R
- added R16: 1k, symbol Device:R
- added SW1: RotaryEncoder, Rotary_Encoder:RotaryEncoder_Alps_EC12E_Vertical_H20mm, symbol Device:RotaryEncoder
- added TP13: XIN, symbol Connector:TestPoint
- added TP14: XOUT, symbol Connector:TestPoint
- added TP15: QSPI_SCLK, symbol Connector:TestPoint
- added TP16: QSPI_SS, symbol Connector:TestPoint
- added TP17: QSPI_SD0, symbol Connector:TestPoint
- added TP18: QSPI_SD1, symbol Connector:TestPoint
- added TP19: QSPI_SD2, symbol Connector:TestPoint
- added TP20: QSPI_SD3, symbol Connector:TestPoint
- added TP21: USB_DP, symbol Connector:TestPoint
- added TP22: USB_DM, symbol Connector:TestPoint
- added TP23: RUN, symbol Connector:TestPoint
- added TP24: DVDD, symbol Connector:TestPoint
- added TP25: IOVDD, symbol Connector:TestPoint
- added TP26: VREG_IN, symbol Connector:TestPoint
- added TP27: SBU1, symbol Connector:TestPoint
- added TP28: SBU2, symbol Connector:TestPoint
- added TP29: CC1, symbol Connector:TestPoint
- added TP30: CC2, symbol Connector:TestPoint
- added TP31: EXP5_INT, symbol Connector:TestPoint
- added TP32: EXP4_INT, symbol Connector:TestPoint
- added TP33: EXP3_INT, symbol Connector:TestPoint
- added TP34: EXP2_INT, symbol Connector:TestPoint
- added TP35: EXP1_INT, symbol Connector:TestPoint
- added TP36: ENC_A, symbol Connector:TestPoint
- added TP37: ENC_B, symbol Connector:TestPoint
- added TP39: NPIXEL_SHIFT, symbol Connector:TestPoint
- added TP40: NPIXEL_IN, symbol Connector:TestPoint
- added U6, U7, U8, U9: PCA9555PW, Package_SO:TSSOP-24_4.4x7.8mm_P0.65mm, symbol Interface_Expansion:PCA9555PW
- MX10, MX11, MX12, MX13, MX14, MX15, MX16, MX17, MX18, MX19, MX2, MX20, MX21, MX22, MX23, MX24, MX25, MX26, MX27, MX28, MX29, MX3, MX30, MX31, MX32, MX33, MX34, MX35, MX36, MX37, MX38, MX39, MX4, MX40, MX41, MX42, MX43, MX44, MX45, MX46, MX47, MX48, MX49, MX5, MX50, MX51, MX52, MX53, MX54, MX55, MX56, MX57, MX58, MX59, MX6, MX60, MX61, MX62, MX63, MX64, MX65, MX66, MX67, MX68, MX69, MX7, MX70, MX71, MX72, MX73, MX74, MX75, MX8, MX9: value MX_SW_HS -> SW_MX_CHOC; footprint CustomKeyboardLibrary:SW_MX_HS_CPG151101S11_1u_Custom -> CustomKeyboardLibrary:SW_choc_mx_combined
- U3: footprint CustomKeyboardLibrary:SN74AHCT125PWR -> PW14; symbol SN74AHCT125PWR:SN74AHCT125PWR -> CustomSymbols:SN74AHCT125PWR
Connections:
- net I2C_1.SCL is gone; now on net I2C1_SCL: J1.3 (Pin_3)
- net I2C_1.SDA is gone; now on net I2C1_SDA: J1.4 (Pin_4)
- net PixelShiftInput is gone; now on net NEOPIXEL_SHIFTER_INPUT: U3.2 (1A)
- net +1V1: now also TP24.1
- net +3V3: now also C86.1, C87.1, C88.1, C89.1, C90.1, R10.1, R11.1, R4.1, R5.1, R9.1, TP25.1, TP26.1, U6.21 (A0), U6.24 (VDD), U7.2 (A1), U7.24 (VDD), U8.2 (A1), U8.21 (A0), U8.24 (VDD), U9.24 (VDD), U9.3 (A2)
- net +5V: now also BZ1.1 (+), C1.2, C10.2, C11.2, C12.2, C13.2, C14.2, C15.2, C16.2, C17.2, C18.2, C19.2, C2.2, C20.2, C21.2, C22.2, C23.2, C24.2, C25.2, C26.2, C27.2, C28.2, C29.2, C3.2, C30.2, C31.2, C32.2, C33.2, C34.2, C35.2, C36.2, C37.2, C38.2, C39.2, C4.2, C40.2, C41.2, C42.2, C43.2, C44.2, C45.2, C46.2, C47.2, C48.2, C49.2, C5.2, C50.2, C51.2, C52.2, C53.2, C54.2, C55.2, C56.2, C57.2, C58.2, C59.2, C6.2, C60.2, C61.2, C62.2, C63.2, C64.2, C65.2, C66.2, C67.2, C68.2, C69.2, C7.2, C70.2, C71.2, C72.2, C73.2, C74.2, C75.2, C8.2, C80.2, C9.2, C91.1, J2.A4 (VBUS), J2.A9 (VBUS), J2.B4 (VBUS), J2.B9 (VBUS), LED76.1 (VDD)
- net GND: now also MX10.1, MX11.1, MX12.1, MX13.1, MX14.1, MX15.1, MX16.1, MX17.1, MX18.1, MX19.1, MX2.1, MX20.1, MX21.1, MX22.1, MX23.1, MX24.1, MX25.1, MX26.1, MX27.1, MX28.1, MX29.1, MX3.1, MX30.1, MX31.1, MX32.1, MX33.1, MX34.1, MX35.1, MX36.1, MX37.1, MX38.1, MX39.1, MX4.1, MX40.1, MX41.1, MX42.1, MX43.1, MX44.1, MX45.1, MX46.1, MX47.1, MX48.1, MX49.1, MX5.1, MX50.1, MX51.1, MX52.1, MX53.1, MX54.1, MX55.1, MX56.1, MX57.1, MX58.1, MX59.1, MX6.1, MX60.1, MX61.1, MX62.1, MX63.1, MX64.1, MX65.1, MX66.1, MX67.1, MX68.1, MX69.1, MX7.1, MX70.1, MX71.1, MX72.1, MX73.1, MX74.1, MX75.1, MX8.1, MX9.1, C1.1, C10.1, C11.1, C12.1, C13.1, C14.1, C15.1, C16.1, C17.1, C18.1, C19.1, C2.1, C20.1, C21.1, C22.1, C23.1, C24.1, C25.1, C26.1, C27.1, C28.1, C29.1, C3.1, C30.1, C31.1, C32.1, C33.1, C34.1, C35.1, C36.1, C37.1, C38.1, C39.1, C4.1, C40.1, C41.1, C42.1, C43.1, C44.1, C45.1, C46.1, C47.1, C48.1, C49.1, C5.1, C50.1, C51.1, C52.1, C53.1, C54.1, C55.1, C56.1, C57.1, C58.1, C59.1, C6.1, C60.1, C61.1, C62.1, C63.1, C64.1, C65.1, C66.1, C67.1, C68.1, C69.1, C7.1, C70.1, C71.1, C72.1, C73.1, C74.1, C75.1, C8.1, C80.1, C86.2, C87.2, C88.2, C89.2, C9.1, C90.2, C91.2, J2.A1 (GND), J2.A12 (GND), J2.B1 (GND), J2.B12 (GND), J2.S1 (SHIELD), LED76.4 (VSS), MX15.1, Q1.3 (C), R12.2, R13.2, SW1.C, U6.12 (VSS), U6.2 (A1), U6.3 (A2), U7.12 (VSS), U7.21 (A0), U7.3 (A2), U8.12 (VSS), U8.3 (A2), U9.12 (VSS), U9.2 (A1), U9.21 (A0)
- net I2C1_SCL: now also U2.22 (SCL), U6.22 (SCL), U7.22 (SCL), U8.22 (SCL), U9.22 (SCL)
- net I2C1_SDA: now also U2.23 (SDA), U6.23 (SDA), U7.23 (SDA), U8.23 (SDA), U9.23 (SDA)
- net RESET: now also TP23.1
- net USB_DM: now also J2.A7 (D-), J2.B7 (D-), R14.1, TP22.1; no longer U1.46 (USB_DM)
- net USB_DP: now also J2.A6 (D+), J2.B6 (D+), R15.1, TP21.1; no longer U1.47 (USB_DP)
- net at C82.2, U1.20 (XIN), Y1.2: now also TP13.1
- net at R7.1, R8.1, U1.56 (QSPI_SS)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: now also TP16.1
- net at R6.2, U1.21 (XOUT): now also TP14.1
- net BUZZER: now reaches U1.27 (GPIO16)
- net BUZZER: now also R16.1
- net EXPANDER1_INT: now reaches U1.31 (GPIO20)
- net EXPANDER1_INT: now also U2.1 (~{INT}), R4.2, TP35.1
- net EXPANDER2_INT: now reaches U1.32 (GPIO21)
- net EXPANDER2_INT: now also R5.2, TP34.1, U6.1 (~{INT})
- net EXPANDER3_INT: now reaches U1.34 (GPIO22)
- net EXPANDER3_INT: now also R9.2, TP33.1, U7.1 (~{INT})
- net EXPANDER4_INT: now reaches U1.35 (GPIO23)
- net EXPANDER4_INT: now also R10.2, TP32.1, U8.1 (~{INT})
- net EXPANDER5_INT: now reaches U1.36 (GPIO24)
- net EXPANDER5_INT: now also R11.2, TP31.1, U9.1 (~{INT})
- net at U1.51 (QSPI_SD3), U4.7 (IO3): now also TP20.1
- net at U1.52 (QSPI_SCLK), U4.6 (CLK): now also TP15.1
- net at U1.53 (QSPI_SD0), U4.5 (DI(IO0)): now also TP17.1
- net at U1.54 (QSPI_SD2), U4.3 (IO2): now also TP19.1
- net at U1.55 (QSPI_SD1), U4.2 (DO(IO1)): now also TP18.1
- net ENCODER_A: now reaches U1.6 (GPIO4)
- net ENCODER_A: now also SW1.A, TP36.1
- net ENCODER_B: now reaches U1.7 (GPIO5)
- net ENCODER_B: now also SW1.B, TP37.1
- net ENCODER_SW: now reaches U1.8 (GPIO6)
- net NEOPIXEL_SHIFTER_INPUT: now reaches U1.9 (GPIO7)
- net NEOPIXEL_SHIFTER_INPUT: now also TP39.1
- removed net Column1: MX16.2, MX31.2, MX46.2, MX61.2, U2.11 (IO0_7)
- removed net Column10: MX10.2, MX25.2, MX40.2, MX55.2, MX70.2, U2.18 (IO1_5)
- removed net Column11: MX11.2, MX26.2, MX41.2, MX56.2, MX71.2, U2.17 (IO1_4)
- removed net Column12: MX12.2, MX27.2, MX42.2, MX57.2, MX72.2, U2.16 (IO1_3)
- removed net Column13: MX13.2, MX28.2, MX43.2, MX58.2, MX73.2, U2.15 (IO1_2)
- removed net Column14: MX14.2, MX29.2, MX44.2, MX59.2, MX74.2, U2.14 (IO1_1)
- removed net Column15: MX15.2, MX30.2, MX45.2, MX60.2, MX75.2, U2.13 (IO1_0)
- removed net Column2: MX17.2, MX2.2, MX32.2, MX47.2, MX62.2, U2.10 (IO0_6)
- removed net Column3: MX18.2, MX3.2, MX33.2, MX48.2, MX63.2, U2.9 (IO0_5)
- removed net Column4: MX19.2, MX34.2, MX4.2, MX49.2, MX64.2, U2.8 (IO0_4)
- removed net Column5: MX20.2, MX35.2, MX5.2, MX50.2, MX65.2, U2.4 (IO0_0)
- removed net Column6: MX21.2, MX36.2, MX51.2, MX6.2, MX66.2, U2.5 (IO0_1)
- removed net Column7: MX22.2, MX37.2, MX52.2, MX67.2, MX7.2, U2.6 (IO0_2)
- removed net Column8: MX23.2, MX38.2, MX53.2, MX68.2, MX8.2, U2.7 (IO0_3)
- removed net Column9: MX24.2, MX39.2, MX54.2, MX69.2, MX9.2, U2.19 (IO1_6)
- net PixelBarInput renamed ENCODER_LED
- net ENCODER_LED: now also LED76.3 (DIN)
- net PixelInput renamed NEOPIXEL_INPUT
- net NEOPIXEL_INPUT: now also TP40.1
- new net: J2.A5 (CC1), R12.1, TP29.1
- new net: Q1.1 (B), R16.2
- new net: R15.2, U1.47 (USB_DP)
- new net: J2.A8 (SBU1), TP27.1
- new net: J2.B5 (CC2), R13.1, TP30.1
- new net: J2.B8 (SBU2), TP28.1
- new net: R14.2, U1.46 (USB_DM)
- new net: BZ1.2 (-), Q1.2 (E)
- new net KEY1: MX15.2, U2.4 (IO0_0)
- new net KEY10: MX10.2, U2.14 (IO1_1)
- new net KEY11: MX11.2, U2.15 (IO1_2)
- new net KEY12: MX12.2, U2.16 (IO1_3)
- new net KEY13: MX13.2, U2.17 (IO1_4)
- new net KEY14: MX14.2, U2.18 (IO1_5)
- new net KEY15: MX15.2, U2.19 (IO1_6)
- new net KEY16: MX16.2, U6.4 (IO0_0)
- new net KEY17: MX17.2, U6.5 (IO0_1)
- new net KEY18: MX18.2, U6.6 (IO0_2)
- new net KEY19: MX19.2, U6.7 (IO0_3)
- new net KEY2: MX2.2, U2.5 (IO0_1)
- new net KEY20: MX20.2, U6.8 (IO0_4)
- new net KEY21: MX21.2, U6.9 (IO0_5)
- new net KEY22: MX22.2, U6.10 (IO0_6)
- new net KEY23: MX23.2, U6.11 (IO0_7)
- new net KEY24: MX24.2, U6.13 (IO1_0)
- new net KEY25: MX25.2, U6.14 (IO1_1)
- new net KEY26: MX26.2, U6.15 (IO1_2)
- new net KEY27: MX27.2, U6.16 (IO1_3)
- new net KEY28: MX28.2, U6.17 (IO1_4)
- new net KEY29: MX29.2, U6.18 (IO1_5)
- new net KEY3: MX3.2, U2.6 (IO0_2)
- new net KEY30: MX30.2, U6.19 (IO1_6)
- new net KEY31: MX31.2, U7.4 (IO0_0)
- new net KEY32: MX32.2, U7.5 (IO0_1)
- new net KEY33: MX33.2, U7.6 (IO0_2)
- new net KEY34: MX34.2, U7.7 (IO0_3)
- new net KEY35: MX35.2, U7.8 (IO0_4)
- new net KEY36: MX36.2, U7.9 (IO0_5)
- new net KEY37: MX37.2, U7.10 (IO0_6)
- new net KEY38: MX38.2, U7.11 (IO0_7)
- new net KEY39: MX39.2, U7.13 (IO1_0)
- new net KEY4: MX4.2, U2.7 (IO0_3)
- new net KEY40: MX40.2, U7.14 (IO1_1)
- new net KEY41: MX41.2, U7.15 (IO1_2)
- new net KEY42: MX42.2, U7.16 (IO1_3)
- new net KEY43: MX43.2, U7.17 (IO1_4)
- new net KEY44: MX44.2, U7.18 (IO1_5)
- new net KEY45: MX45.2, U7.19 (IO1_6)
- new net KEY46: MX46.2, U8.4 (IO0_0)
- new net KEY47: MX47.2, U8.5 (IO0_1)
- new net KEY48: MX48.2, U8.6 (IO0_2)
- new net KEY49: MX49.2, U8.7 (IO0_3)
- new net KEY5: MX5.2, U2.8 (IO0_4)
- new net KEY50: MX50.2, U8.8 (IO0_4)
- new net KEY51: MX51.2, U8.9 (IO0_5)
- new net KEY52: MX52.2, U8.10 (IO0_6)
- new net KEY53: MX53.2, U8.11 (IO0_7)
- new net KEY54: MX54.2, U8.13 (IO1_0)
- new net KEY55: MX55.2, U8.14 (IO1_1)
- new net KEY56: MX56.2, U8.15 (IO1_2)
- new net KEY57: MX57.2, U8.16 (IO1_3)
- new net KEY58: MX58.2, U8.17 (IO1_4)
- new net KEY59: MX59.2, U8.18 (IO1_5)
- new net KEY6: MX6.2, U2.9 (IO0_5)
- new net KEY60: MX60.2, U8.19 (IO1_6)
- new net KEY61: MX61.2, U9.4 (IO0_0)
- new net KEY62: MX62.2, U9.5 (IO0_1)
- new net KEY63: MX63.2, U9.6 (IO0_2)
- new net KEY64: MX64.2, U9.7 (IO0_3)
- new net KEY65: MX65.2, U9.8 (IO0_4)
- new net KEY66: MX66.2, U9.9 (IO0_5)
- new net KEY67: MX67.2, U9.10 (IO0_6)
- new net KEY68: MX68.2, U9.11 (IO0_7)
- new net KEY69: MX69.2, U9.13 (IO1_0)
- new net KEY7: MX7.2, U2.10 (IO0_6)
- new net KEY70: MX70.2, U9.14 (IO1_1)
- new net KEY71: MX71.2, U9.15 (IO1_2)
- new net KEY72: MX72.2, U9.16 (IO1_3)
- new net KEY73: MX73.2, U9.17 (IO1_4)
- new net KEY74: MX74.2, U9.18 (IO1_5)
- new net KEY75: MX75.2, U9.19 (IO1_6)
- new net KEY8: MX8.2, U2.11 (IO0_7)
- new net KEY9: MX9.2, U2.13 (IO1_0)
- no-connect marks 0 -> 33
Other:
- note added: "Accessories"
- note added: "Buzzer"
- note added: "I2C OLED"
- note added: "IO Expanders"
- note added: "Keyboard"
- note added: "Keyswitches"
- note added: "Logic level shifter"
- note added: "Neopixels"
- note added: "Rotary Encoder"
- note added: "USB C Receptacle"
- note removed: "Logic Level Shifter"
- company: (none) -> Edward Hesketh
- title: (none) -> The Slab Keyboard
- moved on the sheet: C76, C77, C78, C79, C81, C82, C83, C84, C85, J1, LED1, MX15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

Commit message: feat: rp2350 design mostly complete
Parts:
- removed C82: 12pF, symbol Device:C
- removed C83, C85: 1uF, symbol Device:C
- removed C84: 100nF, symbol Device:C
- removed R15: 27, symbol Device:R
- removed R7: 1k, symbol Device:R
- removed TP13: XIN, symbol Connector:TestPoint
- removed TP17: QSPI_SD0, symbol Connector:TestPoint
- removed TP18: QSPI_SD1, symbol Connector:TestPoint
- removed TP19: QSPI_SD2, symbol Connector:TestPoint
- removed TP21: USB_DP, symbol Connector:TestPoint
- removed TP22: USB_DM, symbol Connector:TestPoint
- removed TP23: RUN, symbol Connector:TestPoint
- removed TP26: VREG_IN, symbol Connector:TestPoint
- removed U1: RP2040, Package_DFN_QFN:QFN-56-1EP_7x7mm_P0.4mm_EP3.2x3.2mm, symbol MCU_RaspberryPi:RP2040
- removed U5: AP2112K-3.3, Package_TO_SOT_SMD:SOT-23-5, symbol Regulator_Linear:AP2112K-3.3
- removed Y1: 12MHz, symbol Device:Crystal
- added C100, C101: 15pF, Capacitor_SMD:C_0402_1005Metric, symbol Device:C
- added C103, C105, C106, C107, C108, C109, C110, C112, C80, C99: 100nF, Capacitor_SMD:C_0402_1005Metric, symbol Device:C
- added C111: 10u, Capacitor_SMD:C_0805_2012Metric, symbol Device:C
- added C96: 4.7uF, Capacitor_SMD:C_0402_1005Metric, symbol Device:C
- added C97, C98: 4.7uF, RP2350_80QFN_minimal:C_0402_1005Metric_small_pads, symbol Device:C
- added L1: 3.3u, RP2350_80QFN_minimal:L_pol_2016, symbol Device:L
- added R1: 33, Resistor_SMD:R_0402_1005Metric, symbol Device:R
- added R12: DNF, Resistor_SMD:R_0402_1005Metric, symbol Device:R
- added R13: 10k, Resistor_SMD:R_0402_1005Metric, symbol Device:R
- added TP1: 3V3, symbol Connector:TestPoint
- added TP10: QSPI_SS, symbol Connector:TestPoint
- added TP11: QSPI_SD1, symbol Connector:TestPoint
- added TP2: 1V1, symbol Connector:TestPoint
- added TP27: VBUS, symbol Connector:TestPoint
- added TP3: USB_DP, symbol Connector:TestPoint
- added TP4: USB_DM, symbol Connector:TestPoint
- added TP8: QSPI_SD0, symbol Connector:TestPoint
- added U1: NCP1117-3.3_SOT223, Package_TO_SOT_SMD:SOT-223-3_TabPin2, symbol Regulator_Linear:NCP1117-3.3_SOT223
- added U3: RP2350_80QFN, RP2350_80QFN_minimal:RP2350-QFN-80-1EP_10x10_P0.4mm_EP3.4x3.4mm_ThermalVias, symbol RP2350:RP2350_80QFN
- added Y1: ABM8-272-T3, Crystal:Crystal_SMD_3225-4Pin_3.2x2.5mm, symbol Device:Crystal_GND24
- C76, C77: value 100nF -> 10uF; footprint (none) -> Capacitor_SMD:C_0805_2012Metric
- C78: footprint (none) -> Capacitor_SMD:C_0402_1005Metric
- C79: value 100nF -> 4.7uF; footprint (none) -> Capacitor_SMD:C_0402_1005Metric
- C81: value 12pF -> 100nF; footprint (none) -> Capacitor_SMD:C_0402_1005Metric
- R14: value 27 -> 1k; footprint (none) -> Resistor_SMD:R_0402_1005Metric
- R3: value 10k -> 27; footprint (none) -> Resistor_SMD:R_0402_1005Metric
- R6: value 1k -> 27; footprint (none) -> Resistor_SMD:R_0402_1005Metric
- R8: value 10k -> 1k; footprint (none) -> Resistor_SMD:R_0402_1005Metric
- TP14: value XOUT -> QSPI_SCLK
- TP15: value QSPI_SCLK -> QSPI_SD2
- TP16: value QSPI_SS -> QSPI_SD3
- TP20: value QSPI_SD3 -> RUN
- TP24: value DVDD -> XIN
- TP25: value IOVDD -> XOUT
- renumbered C80 to C102, R12 to R15, R13 to R17, R1 to R2, R2 to R7, SW3 to SW2, SW2 to SW3, TP5 to TP12, TP6 to TP13, TP7 to TP17, TP8 to TP18, TP9 to TP19, TP10 to TP21, TP11 to TP22, TP12 to TP23, TP39 to TP26, TP40 to TP28, TP27 to TP38, TP28 to TP39, TP1 to TP5, TP2 to TP6, TP3 to TP7, TP4 to TP9, U3 to U5
Connections:
- net +1V1: now also C78.1, C79.1, C80.1, C98.1, L1.1, TP2.1, U3.10 (DVDD), U3.32 (DVDD), U3.51 (DVDD), U3.65 (VREG_FB); no longer TP24.1
- net +3V3: now also C77.1, C81.2, C103.2, C105.2, C106.2, C107.2, C108.2, C109.2, C110.2, C111.1, C112.2, C97.1, C99.1, R1.1, R12.1, R13.2, TP1.1, U1.2 (VO), U3.15 (IOVDD), U3.24 (IOVDD), U3.29 (IOVDD), U3.41 (IOVDD), U3.5 (IOVDD), U3.50 (IOVDD), U3.59 (ADC_AVDD), U3.60 (IOVDD), U3.64 (VREG_VIN), U3.68 (USB_OTP_VDD), U3.69 (QSPI_IOVDD), U3.76 (IOVDD); no longer C76.1, C78.1, C79.1, R3.1, R8.2, TP25.1
- net +5V: no longer BZ1.1 (+), C1.2, C10.2, C102.2, C11.2, C12.2, C13.2, C14.2, C15.2, C16.2, C17.2, C18.2, C19.2, C2.2, C20.2, C21.2, C22.2, C23.2, C24.2, C25.2, C26.2, C27.2, C28.2, C29.2, C3.2, C30.2, C31.2, C32.2, C33.2, C34.2, C35.2, C36.2, C37.2, C38.2, C39.2, C4.2, C40.2, C41.2, C42.2, C43.2, C44.2, C45.2, C46.2, C47.2, C48.2, C49.2, C5.2, C50.2, C51.2, C52.2, C53.2, C54.2, C55.2, C56.2, C57.2, C58.2, C59.2, C6.2, C60.2, C61.2, C62.2, C63.2, C64.2, C65.2, C66.2, C67.2, C68.2, C69.2, C7.2, C70.2, C71.2, C72.2, C73.2, C74.2, C75.2, C77.1, C8.2, C9.2, C91.1, J2.A4 (VBUS), J2.A9 (VBUS), J2.B4 (VBUS), J2.B9 (VBUS), LED1.1 (VDD), LED10.1 (VDD), LED11.1 (VDD), LED12.1 (VDD), LED13.1 (VDD), LED14.1 (VDD), LED15.1 (VDD), LED16.1 (VDD), LED17.1 (VDD), LED18.1 (VDD), LED19.1 (VDD), LED2.1 (VDD), LED20.1 (VDD), LED21.1 (VDD), LED22.1 (VDD), LED23.1 (VDD), LED24.1 (VDD), LED25.1 (VDD), LED26.1 (VDD), LED27.1 (VDD), LED28.1 (VDD), LED29.1 (VDD), LED3.1 (VDD), LED30.1 (VDD), LED31.1 (VDD), LED32.1 (VDD), LED33.1 (VDD), LED34.1 (VDD), LED35.1 (VDD), LED36.1 (VDD), LED37.1 (VDD), LED38.1 (VDD), LED39.1 (VDD), LED4.1 (VDD), LED40.1 (VDD), LED41.1 (VDD), LED42.1 (VDD), LED43.1 (VDD), LED44.1 (VDD), LED45.1 (VDD), LED46.1 (VDD), LED47.1 (VDD), LED48.1 (VDD), LED49.1 (VDD), LED5.1 (VDD), LED50.1 (VDD), LED51.1 (VDD), LED52.1 (VDD), LED53.1 (VDD), LED54.1 (VDD), LED55.1 (VDD), LED56.1 (VDD), LED57.1 (VDD), LED58.1 (VDD), LED59.1 (VDD), LED6.1 (VDD), LED60.1 (VDD), LED61.1 (VDD), LED62.1 (VDD), LED63.1 (VDD), LED64.1 (VDD), LED65.1 (VDD), LED66.1 (VDD), LED67.1 (VDD), LED68.1 (VDD), LED69.1 (VDD), LED7.1 (VDD), LED70.1 (VDD), LED71.1 (VDD), LED72.1 (VDD), LED73.1 (VDD), LED74.1 (VDD), LED75.1 (VDD), LED76.1 (VDD), LED8.1 (VDD), LED9.1 (VDD), U5.14 (VCC)
- net BUZZER: now also U3.16 (GPIO16)
- net ENCODER_A: now also U3.79 (GPIO2)
- net ENCODER_B: now also U3.80 (GPIO3)
- net EXPANDER1_INT: now also U3.4 (GPIO7)
- net EXPANDER2_INT: now also U3.6 (GPIO8)
- net EXPANDER3_INT: now also U3.7 (GPIO9)
- net EXPANDER4_INT: now also U3.8 (GPIO10)
- net EXPANDER5_INT: now also U3.9 (GPIO11)
- net GND: now also C100.2, C101.2, C103.1, C105.1, C106.1, C107.1, C108.1, C109.1, C110.1, C111.2, C112.1, C80.2, C96.2, C97.2, C98.2, C99.2, U1.1 (GND), U3.62 (VREG_PGND), U3.81 (GND), Y1.2, Y1.4
- net I2C1_SCL: now also U3.2 (GPIO5)
- net I2C1_SDA: now also U3.1 (GPIO4)
- net KEY1: no longer U2.4 (IO0_0)
- net KEY10: no longer U2.14 (IO1_1)
- net KEY11: no longer U2.15 (IO1_2)
- net KEY12: no longer U2.16 (IO1_3)
- net KEY13: no longer U2.17 (IO1_4)
- net KEY14: no longer U2.18 (IO1_5)
- net KEY15: no longer U2.19 (IO1_6)
- net KEY16: no longer U6.4 (IO0_0)
- net KEY17: no longer U6.5 (IO0_1)
- net KEY18: no longer U6.6 (IO0_2)
- net KEY19: no longer U6.7 (IO0_3)
- net KEY2: no longer U2.5 (IO0_1)
- net KEY20: no longer U6.8 (IO0_4)
- net KEY21: no longer U6.9 (IO0_5)
- net KEY22: no longer U6.10 (IO0_6)
- net KEY23: no longer U6.11 (IO0_7)
- net KEY24: no longer U6.13 (IO1_0)
- net KEY25: no longer U6.14 (IO1_1)
- net KEY26: no longer U6.15 (IO1_2)
- net KEY27: no longer U6.16 (IO1_3)
- net KEY28: no longer U6.17 (IO1_4)
- net KEY29: no longer U6.18 (IO1_5)
- net KEY3: no longer U2.6 (IO0_2)
- net KEY30: no longer U6.19 (IO1_6)
- net KEY31: no longer U7.4 (IO0_0)
- net KEY32: no longer U7.5 (IO0_1)
- net KEY33: no longer U7.6 (IO0_2)
- net KEY34: no longer U7.7 (IO0_3)
- net KEY35: no longer U7.8 (IO0_4)
- net KEY36: no longer U7.9 (IO0_5)
- net KEY37: no longer U7.10 (IO0_6)
- net KEY38: no longer U7.11 (IO0_7)
- net KEY39: no longer U7.13 (IO1_0)
- net KEY4: no longer U2.7 (IO0_3)
- net KEY40: no longer U7.14 (IO1_1)
- net KEY41: no longer U7.15 (IO1_2)
- net KEY42: no longer U7.16 (IO1_3)
- net KEY43: no longer U7.17 (IO1_4)
- net KEY44: no longer U7.18 (IO1_5)
- net KEY45: no longer U7.19 (IO1_6)
- net KEY46: no longer U8.4 (IO0_0)
- net KEY47: no longer U8.5 (IO0_1)
- net KEY48: no longer U8.6 (IO0_2)
- net KEY49: no longer U8.7 (IO0_3)
- net KEY5: no longer U2.8 (IO0_4)
- net KEY50: no longer U8.8 (IO0_4)
- net KEY51: no longer U8.9 (IO0_5)
- net KEY52: no longer U8.10 (IO0_6)
- net KEY53: no longer U8.11 (IO0_7)
- net KEY54: no longer U8.13 (IO1_0)
- net KEY55: no longer U8.14 (IO1_1)
- net KEY56: no longer U8.15 (IO1_2)
- net KEY57: no longer U8.16 (IO1_3)
- net KEY58: no longer U8.17 (IO1_4)
- net KEY59: no longer U8.18 (IO1_5)
- net KEY6: no longer U2.9 (IO0_5)
- net KEY60: no longer U8.19 (IO1_6)
- net KEY61: no longer U9.4 (IO0_0)
- net KEY62: no longer U9.5 (IO0_1)
- net KEY63: no longer U9.6 (IO0_2)
- net KEY64: no longer U9.7 (IO0_3)
- net KEY65: no longer U9.8 (IO0_4)
- net KEY66: no longer U9.9 (IO0_5)
- net KEY67: no longer U9.10 (IO0_6)
- net KEY68: no longer U9.11 (IO0_7)
- net KEY69: no longer U9.13 (IO1_0)
- net KEY7: no longer U2.10 (IO0_6)
- net KEY70: no longer U9.14 (IO1_1)
- net KEY71: no longer U9.15 (IO1_2)
- net KEY72: no longer U9.16 (IO1_3)
- net KEY73: no longer U9.17 (IO1_4)
- net KEY74: no longer U9.18 (IO1_5)
- net KEY75: no longer U9.19 (IO1_6)
- net KEY8: no longer U2.11 (IO0_7)
- net KEY9: no longer U2.13 (IO1_0)
- net NEOPIXEL_SHIFTER_INPUT: now also U3.3 (GPIO6)
- net RESET: now also TP20.1, R13.1, U3.35 (RUN); no longer R3.2
- net UART0_RX: now also U3.78 (GPIO1)
- net UART0_TX: now also U3.77 (GPIO0)
- net USB_DM: no longer R14.1
- net QSPI_SCLK: now reaches U4.6 (CLK)
- net QSPI_SCLK: now also TP14.1, U3.71 (QSPI_SCLK); no longer TP15.1
- net QSPI_SD3: now reaches U4.7 (IO3)
- net QSPI_SD3: now also TP16.1, U3.70 (QSPI_SD3); no longer TP20.1
- net at R14.2: now also C101.1, Y1.3
- net QSPI_SD1: now reaches U4.2 (DO(IO1))
- net QSPI_SD1: now also TP11.1, U3.74 (QSPI_SD1)
- net QSPI_SS: now reaches R8.1, U4.1 (~{CS})
- net QSPI_SS: now also R12.2, TP10.1, U3.75 (QSPI_SS); no longer TP16.1
- net SWD: now reaches TP6.1
- net SWD: now also U3.34 (SWD)
- net QSPI_SD0: now reaches U4.5 (DI(IO0))
- net QSPI_SD0: now also TP8.1, U3.72 (QSPI_SD0)
- net USB_D-: now reaches R6.1
- net USB_D-: now also TP4.1; no longer C81.2
- net at R6.2: now also U3.66 (USB_DM); no longer TP14.1
- net SWCLK: now reaches TP5.1
- net SWCLK: now also U3.33 (SWCLK)
- net QSPI_SD2: now reaches U4.3 (IO2)
- net QSPI_SD2: now also TP15.1, U3.73 (QSPI_SD2)
- new net: R14.1, TP25.1, U3.31 (XOUT)
- new net: C100.1, TP24.1, U3.30 (XIN), Y1.1
- new net: R3.2, U3.67 (USB_DP)
- new net USB_D+: R3.1, TP3.1
- new net VBUS: BZ1.1 (+), C1.2, C10.2, C102.2, C11.2, C12.2, C13.2, C14.2, C15.2, C16.2, C17.2, C18.2, C19.2, C2.2, C20.2, C21.2, C22.2, C23.2, C24.2, C25.2, C26.2, C27.2, C28.2, C29.2, C3.2, C30.2, C31.2, C32.2, C33.2, C34.2, C35.2, C36.2, C37.2, C38.2, C39.2, C4.2, C40.2, C41.2, C42.2, C43.2, C44.2, C45.2, C46.2, C47.2, C48.2, C49.2, C5.2, C50.2, C51.2, C52.2, C53.2, C54.2, C55.2, C56.2, C57.2, C58.2, C59.2, C6.2, C60.2, C61.2, C62.2, C63.2, C64.2, C65.2, C66.2, C67.2, C68.2, C69.2, C7.2, C70.2, C71.2, C72.2, C73.2, C74.2, C75.2, C76.1, C8.2, C9.2, C91.1, J2.A4 (VBUS), J2.A9 (VBUS), J2.B4 (VBUS), J2.B9 (VBUS), LED1.1 (VDD), LED10.1 (VDD), LED11.1 (VDD), LED12.1 (VDD), LED13.1 (VDD), LED14.1 (VDD), LED15.1 (VDD), LED16.1 (VDD), LED17.1 (VDD), LED18.1 (VDD), LED19.1 (VDD), LED2.1 (VDD), LED20.1 (VDD), LED21.1 (VDD), LED22.1 (VDD), LED23.1 (VDD), LED24.1 (VDD), LED25.1 (VDD), LED26.1 (VDD), LED27.1 (VDD), LED28.1 (VDD), LED29.1 (VDD), LED3.1 (VDD), LED30.1 (VDD), LED31.1 (VDD), LED32.1 (VDD), LED33.1 (VDD), LED34.1 (VDD), LED35.1 (VDD), LED36.1 (VDD), LED37.1 (VDD), LED38.1 (VDD), LED39.1 (VDD), LED4.1 (VDD), LED40.1 (VDD), LED41.1 (VDD), LED42.1 (VDD), LED43.1 (VDD), LED44.1 (VDD), LED45.1 (VDD), LED46.1 (VDD), LED47.1 (VDD), LED48.1 (VDD), LED49.1 (VDD), LED5.1 (VDD), LED50.1 (VDD), LED51.1 (VDD), LED52.1 (VDD), LED53.1 (VDD), LED54.1 (VDD), LED55.1 (VDD), LED56.1 (VDD), LED57.1 (VDD), LED58.1 (VDD), LED59.1 (VDD), LED6.1 (VDD), LED60.1 (VDD), LED61.1 (VDD), LED62.1 (VDD), LED63.1 (VDD), LED64.1 (VDD), LED65.1 (VDD), LED66.1 (VDD), LED67.1 (VDD), LED68.1 (VDD), LED69.1 (VDD), LED7.1 (VDD), LED70.1 (VDD), LED71.1 (VDD), LED72.1 (VDD), LED73.1 (VDD), LED74.1 (VDD), LED75.1 (VDD), LED76.1 (VDD), LED8.1 (VDD), LED9.1 (VDD), TP27.1, U1.3 (VI), U5.14 (VCC)
- new net VREG_AVDD: C96.1, R1.2, U3.61 (VREG_AVDD)
- new net VREG_LX: L1.2, U3.63 (VREG_LX)
- new net ~{BOOT}: R8.2
- new net ~{KEY10}: U2.14 (IO1_1)
- new net ~{KEY11}: U2.15 (IO1_2)
- new net ~{KEY12}: U2.16 (IO1_3)
- new net ~{KEY13}: U2.17 (IO1_4)
- new net ~{KEY14}: U2.18 (IO1_5)
- new net ~{KEY15}: U2.19 (IO1_6)
- new net ~{KEY16}: U6.4 (IO0_0)
- new net ~{KEY17}: U6.5 (IO0_1)
- new net ~{KEY18}: U6.6 (IO0_2)
- new net ~{KEY19}: U6.7 (IO0_3)
- new net ~{KEY1}: U2.4 (IO0_0)
- new net ~{KEY20}: U6.8 (IO0_4)
- new net ~{KEY21}: U6.9 (IO0_5)
- new net ~{KEY22}: U6.10 (IO0_6)
- new net ~{KEY23}: U6.11 (IO0_7)
- new net ~{KEY24}: U6.13 (IO1_0)
- new net ~{KEY25}: U6.14 (IO1_1)
- new net ~{KEY26}: U6.15 (IO1_2)
- new net ~{KEY27}: U6.16 (IO1_3)
- new net ~{KEY28}: U6.17 (IO1_4)
- new net ~{KEY29}: U6.18 (IO1_5)
- new net ~{KEY2}: U2.5 (IO0_1)
- new net ~{KEY30}: U6.19 (IO1_6)
- new net ~{KEY31}: U7.4 (IO0_0)
- new net ~{KEY32}: U7.5 (IO0_1)
- new net ~{KEY33}: U7.6 (IO0_2)
- new net ~{KEY34}: U7.7 (IO0_3)
- new net ~{KEY35}: U7.8 (IO0_4)
- new net ~{KEY36}: U7.9 (IO0_5)
- new net ~{KEY37}: U7.10 (IO0_6)
- new net ~{KEY38}: U7.11 (IO0_7)
- new net ~{KEY39}: U7.13 (IO1_0)
- new net ~{KEY3}: U2.6 (IO0_2)
- new net ~{KEY40}: U7.14 (IO1_1)
- new net ~{KEY41}: U7.15 (IO1_2)
- new net ~{KEY42}: U7.16 (IO1_3)
- new net ~{KEY43}: U7.17 (IO1_4)
- new net ~{KEY44}: U7.18 (IO1_5)
- new net ~{KEY45}: U7.19 (IO1_6)
- new net ~{KEY46}: U8.4 (IO0_0)
- new net ~{KEY47}: U8.5 (IO0_1)
- new net ~{KEY48}: U8.6 (IO0_2)
- new net ~{KEY49}: U8.7 (IO0_3)
- new net ~{KEY4}: U2.7 (IO0_3)
- new net ~{KEY50}: U8.8 (IO0_4)
- new net ~{KEY51}: U8.9 (IO0_5)
- new net ~{KEY52}: U8.10 (IO0_6)
- new net ~{KEY53}: U8.11 (IO0_7)
- new net ~{KEY54}: U8.13 (IO1_0)
- new net ~{KEY55}: U8.14 (IO1_1)
- new net ~{KEY56}: U8.15 (IO1_2)
- new net ~{KEY57}: U8.16 (IO1_3)
- new net ~{KEY58}: U8.17 (IO1_4)
- new net ~{KEY59}: U8.18 (IO1_5)
- new net ~{KEY5}: U2.8 (IO0_4)
- new net ~{KEY60}: U8.19 (IO1_6)
- new net ~{KEY61}: U9.4 (IO0_0)
- new net ~{KEY62}: U9.5 (IO0_1)
- new net ~{KEY63}: U9.6 (IO0_2)
- new net ~{KEY64}: U9.7 (IO0_3)
- new net ~{KEY65}: U9.8 (IO0_4)
- new net ~{KEY66}: U9.9 (IO0_5)
- new net ~{KEY67}: U9.10 (IO0_6)
- new net ~{KEY68}: U9.11 (IO0_7)
- new net ~{KEY69}: U9.13 (IO1_0)
- new net ~{KEY6}: U2.9 (IO0_5)
- new net ~{KEY70}: U9.14 (IO1_1)
- new net ~{KEY71}: U9.15 (IO1_2)
- new net ~{KEY72}: U9.16 (IO1_3)
- new net ~{KEY73}: U9.17 (IO1_4)
- new net ~{KEY74}: U9.18 (IO1_5)
- new net ~{KEY75}: U9.19 (IO1_6)
- new net ~{KEY7}: U2.10 (IO0_6)
- new net ~{KEY8}: U2.11 (IO0_7)
- new net ~{KEY9}: U2.13 (IO1_0)
- no-connect marks 33 -> 17
Other:
- note added: "128Mb Flash"
- note added: "Main Capacitor"
- note added: "RP2350 Microcontroller"
- note removed: "128MB QSPI Flash"
- note removed: "Accessories"
- note removed: "Crystal Oscillator"
- note removed: "Keyboard"
- note removed: "RP2040"
- moved on the sheet: BZ1, C1, C10, C102, C11, C12, C13, C14, C15, C16, C17, C18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
