File: Slab.kicad_sch (KiCad schematic)
At the start: 328 parts, among them J1 Conn_01x04, J2 USB_C_Receptacle_USB2.0_16P, Q1 MMBT3906, SW1 RotaryEncoder, SW2 SW_Push, SW3 SW_Push, U1 NCP1117-3.3_SOT223, U2 PCA9555PW, U3 RP2350_80QFN, U4 W25Q128JVS, U5 SN74AHCT125PWR, U6 PCA9555PW, U7 PCA9555PW, U8 PCA9555PW, U9 PCA9555PW, Y1 ABM8-272-T3

Commit message: feat: start PCB layout
Parts:
- BZ1: footprint (none) -> Buzzer_Beeper:MagneticBuzzer_CUI_CMT-8504-100-SMT
- C1, C10, C11, C12, C13, C14, C15, C16, C17, C18, C19, C2, C20, C21, C22, C23, C24, C25, C26, C27, C28, C29, C3, C30, C31, C32, C33, C34, C35, C36, C37, C38, C39, C4, C40, C41, C42, C43, C44, C45, C46, C47, C48, C49, C5, C50, C51, C52, C53, C54, C55, C56, C57, C58, C59, C6, C60, C61, C62, C63, C64, C65, C66, C67, C68, C69, C7, C70, C71, C72, C73, C74, C75, C8, C9: footprint (none) -> Capacitor_SMD:C_0402_1005Metric
- C100: renamed from C87; footprint (none) -> Capacitor_SMD:C_0402_1005Metric
- C101: renamed from C88; footprint (none) -> Capacitor_SMD:C_0402_1005Metric
- C102: renamed from C89; footprint (none) -> Capacitor_SMD:C_0402_1005Metric
- C103: renamed from C90; footprint (none) -> Capacitor_SMD:C_0402_1005Metric
- C89: renamed from C97; footprint RP2350_80QFN_minimal:C_0402_1005Metric_small_pads -> CustomKeyboardLibrary:C_0402_1005Metric_small_pads
- C90: renamed from C98; footprint RP2350_80QFN_minimal:C_0402_1005Metric_small_pads -> CustomKeyboardLibrary:C_0402_1005Metric_small_pads
- C94: renamed from C102; footprint (none) -> Capacitor_SMD:C_0402_1005Metric
- C98: renamed from C91; footprint (none) -> Capacitor_SMD:C_0402_1005Metric
- C99: renamed from C86; footprint (none) -> Capacitor_SMD:C_0402_1005Metric
- J1: renamed from J2; footprint (none) -> Connector_USB:USB_C_Receptacle_GCT_USB4105-xx-A_16P_TopMnt_Horizontal
- L1: footprint RP2350_80QFN_minimal:L_pol_2016 -> CustomKeyboardLibrary:L_pol_2016
- LED76: value MX_SK6812MINI-E -> SK6812MINI-E; footprint CustomKeyboardLibrary:LED_MX_6028R-ROT_Custom -> CustomKeyboardLibrary:LED_6028R_Custom
- R12: renamed from R16; footprint (none) -> Resistor_SMD:R_0402_1005Metric
- R13: renamed from R4; footprint (none) -> Resistor_SMD:R_0402_1005Metric
- R14: renamed from R5; footprint (none) -> Resistor_SMD:R_0402_1005Metric
- R15: renamed from R9; footprint (none) -> Resistor_SMD:R_0402_1005Metric
- R16: renamed from R10; footprint (none) -> Resistor_SMD:R_0402_1005Metric
- R17: renamed from R11; footprint (none) -> Resistor_SMD:R_0402_1005Metric
- R7: renamed from R15; footprint (none) -> CustomKeyboardLibrary:SN74AHCT125PWR
- R8: renamed from R17; footprint (none) -> Resistor_SMD:R_0402_1005Metric
- SW1: renamed from SW2; footprint (none) -> Button_Switch_SMD:SW_Push_1P1T_XKB_TS-1187A
- SW2: renamed from SW3; footprint (none) -> Button_Switch_SMD:SW_Push_1P1T_XKB_TS-1187A
- TP1: renamed from TP2; footprint (none) -> TestPoint:TestPoint_Pad_1.0x1.0mm
- TP10: renamed from TP9; footprint (none) -> TestPoint:TestPoint_Pad_1.0x1.0mm
- TP11: renamed from TP1; footprint (none) -> TestPoint:TestPoint_Pad_1.0x1.0mm
- TP12, TP13, TP35: footprint (none) -> TestPoint:TestPoint_Pad_1.0x1.0mm
- TP14: renamed from TP26; footprint (none) -> TestPoint:TestPoint_Pad_1.0x1.0mm
- TP15: renamed from TP17; footprint (none) -> TestPoint:TestPoint_Pad_1.0x1.0mm
- TP16: renamed from TP28; footprint (none) -> TestPoint:TestPoint_Pad_1.0x1.0mm
- TP17: renamed from TP18; footprint (none) -> TestPoint:TestPoint_Pad_1.0x1.0mm
- TP18: renamed from TP19; footprint (none) -> TestPoint:TestPoint_Pad_1.0x1.0mm
- TP19: renamed from TP21; footprint (none) -> TestPoint:TestPoint_Pad_1.0x1.0mm
- TP2: renamed from TP3; footprint (none) -> TestPoint:TestPoint_Pad_1.0x1.0mm
- TP20: renamed from TP22; footprint (none) -> TestPoint:TestPoint_Pad_1.0x1.0mm
- TP21: renamed from TP27; footprint (none) -> TestPoint:TestPoint_Pad_1.0x1.0mm
- TP22: renamed from TP23; footprint (none) -> TestPoint:TestPoint_Pad_1.0x1.0mm
- TP23: renamed from TP29; footprint (none) -> TestPoint:TestPoint_Pad_1.0x1.0mm
- TP24: renamed from TP30; footprint (none) -> TestPoint:TestPoint_Pad_1.0x1.0mm
- TP25: renamed from TP8; footprint (none) -> TestPoint:TestPoint_Pad_1.0x1.0mm
- TP26: renamed from TP10; footprint (none) -> TestPoint:TestPoint_Pad_1.0x1.0mm
- TP27: renamed from TP11; footprint (none) -> TestPoint:TestPoint_Pad_1.0x1.0mm
- TP28: renamed from TP38; footprint (none) -> TestPoint:TestPoint_Pad_1.0x1.0mm
- TP29: renamed from TP39; footprint (none) -> TestPoint:TestPoint_Pad_1.0x1.0mm
- TP3: renamed from TP4; footprint (none) -> TestPoint:TestPoint_Pad_1.0x1.0mm
- TP30: renamed from TP14; footprint (none) -> TestPoint:TestPoint_Pad_1.0x1.0mm
- TP31: renamed from TP15; footprint (none) -> TestPoint:TestPoint_Pad_1.0x1.0mm
- TP32: renamed from TP16; footprint (none) -> TestPoint:TestPoint_Pad_1.0x1.0mm
- TP33: renamed from TP36; footprint (none) -> TestPoint:TestPoint_Pad_1.0x1.0mm
- TP34: renamed from TP37; footprint (none) -> TestPoint:TestPoint_Pad_1.0x1.0mm
- TP36: renamed from TP34; footprint (none) -> TestPoint:TestPoint_Pad_1.0x1.0mm
- TP37: renamed from TP33; footprint (none) -> TestPoint:TestPoint_Pad_1.0x1.0mm
- TP38: renamed from TP32; footprint (none) -> TestPoint:TestPoint_Pad_1.0x1.0mm
- TP39: renamed from TP31; footprint (none) -> TestPoint:TestPoint_Pad_1.0x1.0mm
- TP4: renamed from TP24; footprint (none) -> TestPoint:TestPoint_Pad_1.0x1.0mm
- TP5: renamed from TP25; footprint (none) -> TestPoint:TestPoint_Pad_1.0x1.0mm
- TP6: renamed from TP20; footprint (none) -> TestPoint:TestPoint_Pad_1.0x1.0mm
- TP7: renamed from TP5; footprint (none) -> TestPoint:TestPoint_Pad_1.0x1.0mm
- TP8: renamed from TP6; footprint (none) -> TestPoint:TestPoint_Pad_1.0x1.0mm
- TP9: renamed from TP7; footprint (none) -> TestPoint:TestPoint_Pad_1.0x1.0mm
- U1: renamed from U3; footprint RP2350_80QFN_minimal:RP2350-QFN-80-1EP_10x10_P0.4mm_EP3.4x3.4mm_ThermalVias -> CustomKeyboardLibrary:RP2350-QFN-80-1EP_10x10_P0.4mm_EP3.4x3.4mm_ThermalVias
- U3: renamed from U5; footprint PW14 -> CustomKeyboardLibrary:SN74AHCT125PWR
- renumbered C78 to C76, C79 to C77, C80 to C78, C81 to C79, C103 to C80, C105 to C81, C106 to C82, C107 to C83, C108 to C84, C109 to C85, C110 to C86, C112 to C87, C96 to C88, C100 to C91, C101 to C92, C111 to C93, C76 to C95, C77 to C96, C99 to C97, R2 to R10, R7 to R11, R3 to R2, R6 to R3, R8 to R4, R14 to R5, R13 to R6, R12 to R9, SW1 to SW3, U1 to U2
Connections:
- net KEY1 is gone; now on net ~{KEY1}: MX15.2

Commit message: feat: layout + track most of board
Parts:
- removed C86: 100nF, Capacitor_SMD:C_0402_1005Metric, symbol Device:C
- removed TP11: 3V3, TestPoint:TestPoint_Pad_1.0x1.0mm, symbol Connector:TestPoint
- removed TP21: VBUS, TestPoint:TestPoint_Pad_1.0x1.0mm, symbol Connector:TestPoint
- removed TP25: QSPI_SD0, TestPoint:TestPoint_Pad_1.0x1.0mm, symbol Connector:TestPoint
- removed TP27: QSPI_SD1, TestPoint:TestPoint_Pad_1.0x1.0mm, symbol Connector:TestPoint
- removed TP28: SBU1, TestPoint:TestPoint_Pad_1.0x1.0mm, symbol Connector:TestPoint
- removed TP29: SBU2, TestPoint:TestPoint_Pad_1.0x1.0mm, symbol Connector:TestPoint
- removed TP30: QSPI_SCLK, TestPoint:TestPoint_Pad_1.0x1.0mm, symbol Connector:TestPoint
- removed TP31: QSPI_SD2, TestPoint:TestPoint_Pad_1.0x1.0mm, symbol Connector:TestPoint
- removed TP32: QSPI_SD3, TestPoint:TestPoint_Pad_1.0x1.0mm, symbol Connector:TestPoint
- removed TP35: EXP1_INT, TestPoint:TestPoint_Pad_1.0x1.0mm, symbol Connector:TestPoint
- removed TP36: EXP2_INT, TestPoint:TestPoint_Pad_1.0x1.0mm, symbol Connector:TestPoint
- removed TP37: EXP3_INT, TestPoint:TestPoint_Pad_1.0x1.0mm, symbol Connector:TestPoint
- removed TP38: EXP4_INT, TestPoint:TestPoint_Pad_1.0x1.0mm, symbol Connector:TestPoint
- removed TP39: EXP5_INT, TestPoint:TestPoint_Pad_1.0x1.0mm, symbol Connector:TestPoint
- removed U1: RP2350_80QFN, CustomKeyboardLibrary:RP2350-QFN-80-1EP_10x10_P0.4mm_EP3.4x3.4mm_ThermalVias, symbol RP2350:RP2350_80QFN
- added MP1, MP10, MP2, MP3, MP4, MP5, MP6, MP7, MP8, MP9: MountingHole_Pad, MountingHole:MountingHole_3.2mm_M3_Pad_TopBottom, symbol Mechanical:MountingHole_Pad
- added RV1: R_Potentiometer, CustomKeyboardLibrary:SW_RS45111A900F_ALPS, symbol Device:R_Potentiometer
- added U1: ADS1110, Package_TO_SOT_SMD:SOT-23-6, symbol Analog_ADC:ADS1110
- added U10: RP2350_60QFN, CustomKeyboardLibrary:RP2350-QFN-60-1EP_7x7_P0.4mm_EP3.4x3.4mm_ThermalVias, symbol RP2350_60:RP2350_60QFN
- C1, C10, C100, C101, C102, C103, C11, C12, C13, C14, C15, C16, C17, C18, C19, C2, C20, C21, C22, C23, C24, C25, C26, C27, C28, C29, C3, C30, C31, C32, C33, C34, C35, C36, C37, C38, C39, C4, C40, C41, C42, C43, C44, C45, C46, C47, C48, C49, C5, C50, C51, C52, C53, C54, C55, C56, C57, C58, C59, C6, C60, C61, C62, C63, C64, C65, C66, C67, C68, C69, C7, C70, C71, C72, C73, C74, C75, C8, C85, C9, C94, C97, C98, C99: footprint Capacitor_SMD:C_0402_1005Metric -> Capacitor_SMD:C_0603_1608Metric_Pad1.08x0.95mm_HandSolder
- MX15, MX16, MX17, MX18, MX19, MX2, MX20, MX21, MX22, MX23, MX24, MX3, MX31, MX32, MX33, MX34, MX35, MX36, MX37, MX4, MX46, MX47, MX48, MX49, MX5, MX50, MX51, MX52, MX53, MX54, MX55, MX6, MX61, MX62, MX63, MX64, MX65, MX66, MX67, MX68, MX69, MX7, MX70, MX71, MX72, MX73, MX74, MX75, MX8: footprint CustomKeyboardLibrary:SW_choc_mx_combined -> CustomKeyboardLibrary:SW_choc_mx_combined_swapped_pads
- R10, R11: footprint Resistor_SMD:R_1206_3216Metric_Pad1.30x1.75mm_HandSolder -> Resistor_SMD:R_0603_1608Metric_Pad0.98x0.95mm_HandSolder
- R12, R13, R14, R15, R16, R17, R8: footprint Resistor_SMD:R_0402_1005Metric -> Resistor_SMD:R_0603_1608Metric_Pad0.98x0.95mm_HandSolder
- R7: footprint CustomKeyboardLibrary:SN74AHCT125PWR -> Resistor_SMD:R_0603_1608Metric_Pad0.98x0.95mm_HandSolder
- TP10, TP12, TP13, TP15, TP17, TP18, TP19, TP20, TP22, TP7, TP8, TP9: footprint TestPoint:TestPoint_Pad_1.0x1.0mm -> Connector_PinHeader_2.54mm:PinHeader_1x01_P2.54mm_Vertical
Connections:
- net +5V is gone; now on net VBUS: TP13.1, TP22.1
- net BOOT is gone; now on net ~{BOOT}: SW2.1
- net KEY10 is gone; now on net ~{KEY10}: MX10.2
- net KEY11 is gone; now on net ~{KEY11}: MX11.2
- net KEY12 is gone; now on net ~{KEY12}: MX12.2
- net KEY13 is gone; now on net ~{KEY13}: MX13.2
- net KEY14 is gone; now on net ~{KEY14}: MX14.2
- net KEY15 is gone; now on net ~{KEY15}: MX15.2
- net KEY16 is gone; now on net ~{KEY16}: MX16.2
- net KEY17 is gone; now on net ~{KEY17}: MX17.2
- net KEY18 is gone; now on net ~{KEY18}: MX18.2
- net KEY19 is gone; now on net ~{KEY19}: MX19.2
- net KEY2 is gone; now on net ~{KEY2}: MX2.2
- net KEY20 is gone; now on net ~{KEY20}: MX20.2
- net KEY21 is gone; now on net ~{KEY21}: MX21.2
- net KEY22 is gone; now on net ~{KEY22}: MX22.2
- net KEY23 is gone; now on net ~{KEY23}: MX23.2
- net KEY24 is gone; now on net ~{KEY24}: MX24.2
- net KEY25 is gone; now on net ~{KEY25}: MX25.2
- net KEY26 is gone; now on net ~{KEY26}: MX26.2
- net KEY27 is gone; now on net ~{KEY27}: MX27.2
- net KEY28 is gone; now on net ~{KEY28}: MX28.2
- net KEY29 is gone; now on net ~{KEY29}: MX29.2
- net KEY3 is gone; now on net ~{KEY3}: MX3.2
- net KEY30 is gone; now on net ~{KEY30}: MX30.2
- net KEY31 is gone; now on net ~{KEY31}: MX31.2
- net KEY32 is gone; now on net ~{KEY32}: MX32.2
- net KEY33 is gone; now on net ~{KEY33}: MX33.2
- net KEY34 is gone; now on net ~{KEY34}: MX34.2
- net KEY35 is gone; now on net ~{KEY35}: MX35.2
- net KEY36 is gone; now on net ~{KEY36}: MX36.2
- net KEY37 is gone; now on net ~{KEY37}: MX37.2
- net KEY38 is gone; now on net ~{KEY38}: MX38.2
- net KEY39 is gone; now on net ~{KEY39}: MX39.2
- net KEY4 is gone; now on net ~{KEY4}: MX4.2
- net KEY40 is gone; now on net ~{KEY40}: MX40.2
- net KEY41 is gone; now on net ~{KEY41}: MX41.2
- net KEY42 is gone; now on net ~{KEY42}: MX42.2
- net KEY43 is gone; now on net ~{KEY43}: MX43.2
- net KEY44 is gone; now on net ~{KEY44}: MX44.2
- net KEY45 is gone; now on net ~{KEY45}: MX45.2
- net KEY46 is gone; now on net ~{KEY46}: MX46.2
- net KEY47 is gone; now on net ~{KEY47}: MX47.2
- net KEY48 is gone; now on net ~{KEY48}: MX48.2
- net KEY49 is gone; now on net ~{KEY49}: MX49.2
- net KEY5 is gone; now on net ~{KEY5}: MX5.2
- net KEY50 is gone; now on net ~{KEY50}: MX50.2
- net KEY51 is gone; now on net ~{KEY51}: MX51.2
- net KEY52 is gone; now on net ~{KEY52}: MX52.2
- net KEY53 is gone; now on net ~{KEY53}: MX53.2
- net KEY54 is gone; now on net ~{KEY54}: MX54.2
- net KEY55 is gone; now on net ~{KEY55}: MX55.2
- net KEY56 is gone; now on net ~{KEY56}: MX56.2
- net KEY57 is gone; now on net ~{KEY57}: MX57.2
- net KEY58 is gone; now on net ~{KEY58}: MX58.2
- net KEY59 is gone; now on net ~{KEY59}: MX59.2
- net KEY6 is gone; now on net ~{KEY6}: MX6.2
- net KEY60 is gone; now on net ~{KEY60}: MX60.2
- net KEY61 is gone; now on net ~{KEY61}: MX61.2
- net KEY62 is gone; now on net ~{KEY62}: MX62.2
- net KEY63 is gone; now on net ~{KEY63}: MX63.2
- net KEY64 is gone; now on net ~{KEY64}: MX64.2
- net KEY65 is gone; now on net ~{KEY65}: MX65.2
- net KEY66 is gone; now on net ~{KEY66}: MX66.2
- net KEY67 is gone; now on net ~{KEY67}: MX67.2
- net KEY68 is gone; now on net ~{KEY68}: MX68.2
- net KEY69 is gone; now on net ~{KEY69}: MX69.2
- net KEY7 is gone; now on net ~{KEY7}: MX7.2
- net KEY70 is gone; now on net ~{KEY70}: MX70.2
- net KEY71 is gone; now on net ~{KEY71}: MX71.2
- net KEY72 is gone; now on net ~{KEY72}: MX72.2
- net KEY73 is gone; now on net ~{KEY73}: MX73.2
- net KEY74 is gone; now on net ~{KEY74}: MX74.2
- net KEY75 is gone; now on net ~{KEY75}: MX75.2
- net KEY8 is gone; now on net ~{KEY8}: MX8.2
- net KEY9 is gone; now on net ~{KEY9}: MX9.2
- net USB_DM is gone; now on net USB_D-: J1.A7 (D-), J1.B7 (D-)
- net USB_DP is gone; now on net USB_D+: J1.A6 (D+), J1.B6 (D+)
- net +1V1: now also U10.23 (DVDD), U10.39 (DVDD), U10.50 (VREG_FB), U10.6 (DVDD)
- net +3V3: now also TP17.1, RV1.1, U1.5 (VDD), U10.1 (IOVDD), U10.11 (IOVDD), U10.20 (IOVDD), U10.30 (IOVDD), U10.38 (IOVDD), U10.44 (ADC_AVDD), U10.45 (IOVDD), U10.49 (VREG_VIN), U10.53 (USB_OTP_VDD), U10.54 (QSPI_IOVDD)
- net BUZZER: now also U10.27 (GPIO16)
- net ENCODER_A: now also U10.4 (GPIO2)
- net ENCODER_B: now also U10.5 (GPIO3)
- net EXPANDER1_INT: now also U10.10 (GPIO7)
- net EXPANDER2_INT: now also U10.12 (GPIO8)
- net EXPANDER3_INT: now also U10.13 (GPIO9)
- net EXPANDER4_INT: now also U10.14 (GPIO10)
- net EXPANDER5_INT: now also U10.15 (GPIO11)
- net GND: now also MP1.1, MP10.1, MP2.1, MP3.1, MP4.1, MP5.1, MP6.1, MP7.1, MP8.1, MP9.1, RV1.3, U1.2 (GND), U1.6 (VIN-), U10.47 (VREG_PGND), U10.61 (GND)
- net I2C1_SCL: now also U1.3 (SCL), U10.8 (GPIO5)
- net I2C1_SDA: now also U1.4 (SDA), U10.7 (GPIO4)
- net NEOPIXEL_SHIFTER_INPUT: now also U10.9 (GPIO6)
- net QSPI_SCLK: now also U10.56 (QSPI_SCLK)
- net QSPI_SD0: now also U10.57 (QSPI_SD0)
- net QSPI_SD1: now also U10.59 (QSPI_SD1)
- net QSPI_SD2: now also U10.58 (QSPI_SD2)
- net QSPI_SD3: now also U10.55 (QSPI_SD3)
- net QSPI_SS: now also U10.60 (QSPI_SS)
- net SWCLK: now also U10.24 (SWCLK)
- net SWD: now also U10.25 (SWD)
- net UART0_RX: now also U10.3 (GPIO1)
- net UART0_TX: now also U10.2 (GPIO0)
- net VREG_AVDD: now also U10.46 (VREG_AVDD)
- net VREG_LX: now also U10.48 (VREG_LX)
- net at R5.1, TP5.1: now also U10.22 (XOUT)
- net at C91.1, TP4.1, Y1.1: now also U10.21 (XIN)
- net at R2.2: now also U10.52 (USB_DP)
- net at R3.2: now also U10.51 (USB_DM)
- net RESET renamed ~{RESET}
- net ~{RESET}: now also U10.26 (RUN)
- new net: RV1.2, U1.1 (VIN+)
- no-connect marks 17 -> 18
Other:
- note added: "Hardware"
- moved on the sheet: C80, C87, C93, R2, R3, TP2, TP3

Commit message: feat: almost fully finished design
Parts:
- removed TP10, TP12, TP13, TP15, TP17, TP18, TP19, TP20, TP22, TP7, TP8, TP9: TestPoint, Connector_PinHeader_2.54mm:PinHeader_1x01_P2.54mm_Vertical, symbol Connector:TestPoint
- added J3, J4: Conn_01x06, Connector_PinHeader_2.54mm:PinHeader_1x06_P2.54mm_Vertical, symbol Connector_Generic:Conn_01x06
- added MP11: MountingHole_Pad, MountingHole:MountingHole_3.2mm_M3_Pad_TopBottom, symbol Mechanical:MountingHole_Pad
Connections:
- net +3V3: now also J4.5 (Pin_5)
- net GND: now also J3.4 (Pin_4), J4.4 (Pin_4), MP11.1
- net I2C1_SCL: now also J4.2 (Pin_2)
- net I2C1_SDA: now also J4.3 (Pin_3)
- net SWCLK: now also J3.6 (Pin_6)
- net SWD: now also J3.5 (Pin_5)
- net UART0_RX: now also J3.2 (Pin_2)
- net UART0_TX: now also J3.3 (Pin_3)
- net VBUS: now also J3.1 (Pin_1), J4.1 (Pin_1)
