File: interchange-connector-test/interchange-connector-test.kicad_sch (KiCad schematic)
At the start: 2 parts, among them U1 MCP2515-xST

Commit message: wip
Parts:
- added U2: SN65HVD1050D, Package_SO:SOIC-8_3.9x4.9mm_P1.27mm, symbol Interface_CAN_LIN:SN65HVD1050D
Other:
- moved on the sheet: A1, U1
Changed lines of the file:
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@@
 	(paper "A4")
 	(symbol
+		(lib_id "Interface_CAN_LIN:SN65HVD1050D")
+		(at 35.56 88.9 0)
+		(unit 1)
+		(body_style 1)
+		(exclude_from_sim no)
+		(in_bom yes)
+		(on_board yes)
+		(in_pos_files yes)
+		(dnp no)
+		(fields_autoplaced yes)
+		(property "Reference" "U2"
+			(at 37.7033 76.2 0)
+			(show_name no)
+			(do_not_autoplace no)
+			(effects
+				(font
+					(size 1.27 1.27)
+				)
+				(justify left)
+			)
+		)
+		(property "Value" "SN65HVD1050D"
+			(at 37.7033 78.74 0)
+			(show_name no)
+			(do_not_autoplace no)
+			(effects
+				(font
+					(size 1.27 1.27)
+				)
+				(justify left)
+			)
+		)
+		(property "Footprint" "Package_SO:SOIC-8_3.9x4.9mm_P1.27mm"
+			(at 35.56 101.6 0)
+			(hide yes)
+			(show_name no)
+			(do_not_autoplace no)
+			(effects
+				(font
+					(size 1.27 1.27)
+				)
+			)
+		)
+		(property "Datasheet" "http://www.ti.com/lit/ds/symlink/sn65hvd1050.pdf"
+			(at 33.02 78.74 0)
+			(hide yes)
+			(show_name no)
+			(do_not_autoplace no)
+			(effects
+				(font
+					(size 1.27 1.27)
+				)
+			)
+		)
+		(property "Description" "CAN Bus Transceiver, EMC optimised, 5.0V, 1Mbps, SOIC-8"
+			(at 35.56 88.9 0)
+			(hide yes)
+			(show_name no)
+			(do_not_autoplace no)
+			(effects
+				(font
+					(size 1.27 1.27)
+				)
+			)
+		)
+		(pin "1"
+		)
+		(pin "2"
+		)
+		(pin "4"
+		)
+		(pin "5"
+		)
+		(pin "6"
+		)
+		(pin "7"
+		)
+		(pin "3"
+		)
+		(pin "8"
+		)
+		(instances
+			(project "interchange-connector-test"
+				(path "/755ae813-dcf9-43a3-8986-d7cb89ce2ddb"
+					(reference "U2")
+					(unit 1)
+				)
+			)
+		)
+	)
+	(symbol
 		(lib_id "MCU_Module:RaspberryPi_Pico")
-		(at 139.7 68.58 0)
+		(at 138.43 96.52 0)
 		(unit 1)
 		(body_style 1)
@@
 		(fields_autoplaced yes)
 		(property "Reference" "A1"
-			(at 141.8433 102.87 0)
+			(at 140.5733 130.81 0)
 			(show_name no)
 			(do_not_autoplace no)
@@
 		)
 		(property "Value" "RaspberryPi_Pico"
-			(at 141.8433 105.41 0)
+			(at 140.5733 133.35 0)
 			(show_name no)
 			(do_not_autoplace no)
@@
 		)
 		(property "Footprint" "Module:RaspberryPi_Pico_Common_THT"
-			(at 139.7 115.57 0)
+			(at 138.43 143.51 0)
 			(hide yes)
 			(show_name no)
@@
 		)
 		(property "Datasheet" "https://datasheets.raspberrypi.com/pico/pico-datasheet.pdf"
-			(at 139.7 118.11 0)
+			(at 138.43 146.05 0)
 			(hide yes)
 			(show_name no)
@@
 		)
 		(property "Description" "Versatile and inexpensive microcontroller module powered by RP2040 dual-core Arm Cortex-M0+ processor up to 133 MHz, 264kB SRAM, 2MB QSPI flash; also supports Raspberry Pi Pico 2"
-			(at 139.7 120.65 0)
+			(at 138.43 148.59 0)
 			(hide yes)
 			(show_name no)
@@
 	(symbol
 		(lib_id "Interface_CAN_LIN:MCP2515-xST")
-		(at 138.43 137.16 0)
+		(at 77.47 95.25 0)
 		(unit 1)
 		(body_style 1)
@@
 		(fields_autoplaced yes)
 		(property "Reference" "U1"
-			(at 140.5733 114.3 0)
+			(at 79.6133 72.39 0)
 			(show_name no)
 			(do_not_autoplace no)
@@
 		)
 		(property "Value" "MCP2515-xST"
-			(at 140.5733 116.84 0)
+			(at 79.6133 74.93 0)
 			(show_name no)
 			(do_not_autoplace no)
@@
 		)
 		(property "Footprint" "Package_SO:TSSOP-20_4.4x6.5mm_P0.65mm"
-			(at 138.43 160.02 0)
+			(at 77.47 118.11 0)
 			(hide yes)
 			(show_name no)
@@
 		)
 		(property "Datasheet" "http://ww1.microchip.com/downloads/en/DeviceDoc/21801e.pdf"
-			(at 140.97 157.48 0)
+			(at 80.01 115.57 0)
 			(hide yes)
 			(show_name no)
@@
 		)
 		(property "Description" "Stand-Alone CAN Controller with SPI Interface, TSSOP-20"
-			(at 138.43 137.16 0)
-			(hide yes)
-			(show_name no)
+			(at 77.47 95.25 0)
+			(hide yes)
+			(show_name no)
